File: KiCad_files/esp.kicad_sch (KiCad schematic)
At the start: 11 parts, among them J2 USB_C_Receptacle_USB2.0_16P, SW1 SW_Push, U1 ESP32-S3-MINI-1U, U2 BNO055

Commit message: tyhjät symboolit
Parts:
- added U3: ~, symbol Projektin osat:BMP581
- added U4: ~, symbol Projektin osat:M20048-1
- added U5: ~, symbol Projektin osat:MP2235S
Other:
- note added: "GNSS moduulin M20048-1 footprinttiä ei löydy peruskirjastosta, en tiiä oisko jossain saatavilla Sama homma IMUn kanssa (BNO055) Sama hakkurin kanssa (MP2235SGJ-Z) Tein niille tyhjät symbolit ja footprintit paikallisiin kirjastoihin, pitää vaan toteuttaa ne:"
- note removed: "GNSS moduulin footprinttiä ei löydy peruskirjastosta, en tiiä oisko jossain saatavilla"
Changed lines of the file:
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@@
 		)
 	)
-	(text "GNSS moduulin footprinttiä ei löydy peruskirjastosta, en tiiä oisko jossain saatavilla"
-		(exclude_from_sim no)
-		(at 151.638 41.91 0)
+	(text "GNSS moduulin M20048-1 footprinttiä ei löydy peruskirjastosta, en tiiä oisko jossain saatavilla\nSama homma IMUn kanssa (BNO055)\nSama hakkurin kanssa (MP2235SGJ-Z)\n\n\nTein niille tyhjät symbolit ja footprintit paikallisiin kirjastoihin, pitää vaan toteuttaa ne:"
+		(exclude_from_sim no)
+		(at 146.05 40.132 0)
 		(effects
 			(font
@@
 	)
 	(symbol
+		(lib_id "Projektin osat:BMP581")
+		(at 121.92 57.15 0)
+		(unit 1)
+		(exclude_from_sim no)
+		(in_bom yes)
+		(on_board yes)
+		(dnp no)
+		(fields_autoplaced yes)
+		(property "Reference" "U3"
+			(at 123.19 55.8799 0)
+			(effects
+				(font
+					(size 1.27 1.27)
+				)
+				(justify left)
+			)
+		)
+		(property "Value" "~"
+			(at 123.19 58.4199 0)
+			(effects
+				(font
+					(size 1.27 1.27)
+				)
+				(justify left)
+			)
+		)
+		(property "Footprint" ""
+			(at 121.92 57.15 0)
+			(effects
+				(font
+					(size 1.27 1.27)
+				)
+				(hide yes)
+			)
+		)
+		(property "Datasheet" ""
+			(at 121.92 57.15 0)
+			(effects
+				(font
+					(size 1.27 1.27)
+				)
+				(hide yes)
+			)
+		)
+		(property "Description" ""
+			(at 121.92 57.15 0)
+			(effects
+				(font
+					(size 1.27 1.27)
+				)
+				(hide yes)
+			)
+		)
+		(instances
+			(project ""
+				(path "/186d5500-054c-4b47-a89c-85f6ce2abe33"
+					(reference "U3")
+					(unit 1)
+				)
+			)
+		)
+	)
+	(symbol
 		(lib_id "power:+3.3V")
 		(at 222.25 190.5 0)
@@
 	)
 	(symbol
+		(lib_id "Projektin osat:MP2235S")
+		(at 161.29 55.88 0)
+		(unit 1)
+		(exclude_from_sim no)
+		(in_bom yes)
+		(on_board yes)
+		(dnp no)
+		(fields_autoplaced yes)
+		(property "Reference" "U5"
+			(at 162.56 54.6099 0)
+			(effects
+				(font
+					(size 1.27 1.27)
+				)
+				(justify left)
+			)
+		)
+		(property "Value" "~"
+			(at 162.56 57.1499 0)
+			(effects
+				(font
+					(size 1.27 1.27)
+				)
+				(justify left)
+			)
+		)
+		(property "Footprint" ""
+			(at 161.29 55.88 0)
+			(effects
+				(font
+					(size 1.27 1.27)
+				)
+				(hide yes)
+			)
+		)
+		(property "Datasheet" ""
+			(at 161.29 55.88 0)
+			(effects
+				(font
+					(size 1.27 1.27)
+				)
+				(hide yes)
+			)
+		)
+		(property "Description" ""
+			(at 161.29 55.88 0)
+			(effects
+				(font
+					(size 1.27 1.27)
+				)
+				(hide yes)
+			)
+		)
+		(instances
+			(project ""
+				(path "/186d5500-054c-4b47-a89c-85f6ce2abe33"
+					(reference "U5")
+					(unit 1)
+				)
+			)
+		)
+	)
+	(symbol
 		(lib_id "Device:R")
 		(at 25.4 262.89 0)
@@
 					(unit 1)
 				)
+			)
+		)
+	)
+	(symbol
+		(lib_id "Projektin osat:M20048-1")
+		(at 140.97 55.88 0)
+		(unit 1)
+		(exclude_from_sim no)
+		(in_bom yes)
+		(on_board yes)
+		(dnp no)
+		(property "Reference" "U4"
+			(at 142.494 53.594 0)
+			(effects
+				(font
+					(size 1.27 1.27)
+				)
+				(justify left)
+			)
+		)
+		(property "Value" "~"
+			(at 142.24 57.1499 0)
+			(effects
+				(font
+					(size 1.27 1.27)
+				)
+				(justify left)
+			)
+		)
+		(property "Footprint" ""
+			(at 140.97 55.88 0)
+			(effects
+				(font
+					(size 1.27 1.27)
+				)
+				(hide yes)
+			)
+		)
+		(property "Datasheet" ""
+			(at 140.97 55.88 0)
+			(effects
+				(font
+					(size 1.27 1.27)
+				)
+				(hide yes)
+			)
+		)
+		(property "Description" ""
+			(at 140.97 55.88 0)
+			(effects
+				(font
+					(size 1.27 1.27)
+				)
+				(hide yes)
+			)
+		)
+		(instances
+			(project ""
+				(path "/186d5500-054c-4b47-a89c-85f6ce2abe33"
+					(reference "U4")
+					(unit 1)
+				)

Commit message: symbolit tehty puuttuville komponenteille
Parts:
- removed U3: ~, symbol Projektin osat:BMP581
- removed U4: ~, symbol Projektin osat:M20048-1
- removed U5: ~, symbol Projektin osat:MP2235S
- added U3: ~, symbol 1_projektin osat:BMP581
- added U4: ~, symbol 1_projektin osat:M20048-1
- added U5: ~, symbol 1_projektin osat:MP2235S
Other:
- note added: "GNSS moduulin M20048-1 footprinttiä ei löydy peruskirjastosta, en tiiä oisko jossain saatavilla Sama homma IMUn kanssa (BNO055) Sama hakkurin kanssa (MP2235SGJ-Z) Tässä symbolit. Footprintit pitää tehdä vielä"
- note removed: "GNSS moduulin M20048-1 footprinttiä ei löydy peruskirjastosta, en tiiä oisko jossain saatavilla Sama homma IMUn kanssa (BNO055) Sama hakkurin kanssa (MP2235SGJ-Z) Tein niille tyhjät symbolit ja footprintit paikallisiin kirjastoihin, pitää vaan toteuttaa ne:"
- moved on the sheet: U2
Changed lines of the file:
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@@
 		)
 	)
-	(text "GNSS moduulin M20048-1 footprinttiä ei löydy peruskirjastosta, en tiiä oisko jossain saatavilla\nSama homma IMUn kanssa (BNO055)\nSama hakkurin kanssa (MP2235SGJ-Z)\n\n\nTein niille tyhjät symbolit ja footprintit paikallisiin kirjastoihin, pitää vaan toteuttaa ne:"
-		(exclude_from_sim no)
-		(at 146.05 40.132 0)
+	(text "GNSS moduulin M20048-1 footprinttiä ei löydy peruskirjastosta, en tiiä oisko jossain saatavilla\nSama homma IMUn kanssa (BNO055)\nSama hakkurin kanssa (MP2235SGJ-Z)\n\n\nTässä symbolit. Footprintit pitää tehdä vielä"
+		(exclude_from_sim no)
+		(at 146.05 43.688 0)
 		(effects
 			(font
@@
 	(symbol
 		(lib_id "Sensor_Motion:BNO055")
-		(at 64.77 64.77 0)
+		(at 64.77 66.04 0)
 		(unit 1)
 		(exclude_from_sim no)
@@
 		(fields_autoplaced yes)
 		(property "Reference" "U2"
-			(at 69.4533 44.45 0)
+			(at 69.4533 45.72 0)
 			(effects
 				(font
@@
 		)
 		(property "Value" "BNO055"
-			(at 69.4533 46.99 0)
+			(at 69.4533 48.26 0)
 			(effects
 				(font
@@
 		)
 		(property "Footprint" "Package_LGA:LGA-28_5.2x3.8mm_P0.5mm"
-			(at 71.12 81.28 0)
+			(at 71.12 82.55 0)
 			(effects
 				(font
@@
 		)
 		(property "Datasheet" "https://www.bosch-sensortec.com/media/boschsensortec/downloads/datasheets/bst-bno055-ds000.pdf"
-			(at 64.77 59.69 0)
+			(at 64.77 60.96 0)
 			(effects
 				(font
@@
 		)
 		(property "Description" "Intelligent 9-axis absolute orientation sensor, LGA-28"
-			(at 64.77 64.77 0)
+			(at 64.77 66.04 0)
 			(effects
 				(font
@@
 	)
 	(symbol
-		(lib_id "Projektin osat:BMP581")
-		(at 121.92 57.15 0)
-		(unit 1)
-		(exclude_from_sim no)
-		(in_bom yes)
-		(on_board yes)
-		(dnp no)
-		(fields_autoplaced yes)
-		(property "Reference" "U3"
-			(at 123.19 55.8799 0)
-			(effects
-				(font
-					(size 1.27 1.27)
-				)
-				(justify left)
-			)
-		)
-		(property "Value" "~"
-			(at 123.19 58.4199 0)
-			(effects
-				(font
-					(size 1.27 1.27)
-				)
-				(justify left)
-			)
-		)
-		(property "Footprint" ""
-			(at 121.92 57.15 0)
-			(effects
-				(font
-					(size 1.27 1.27)
-				)
-				(hide yes)
-			)
-		)
-		(property "Datasheet" ""
-			(at 121.92 57.15 0)
-			(effects
-				(font
-					(size 1.27 1.27)
-				)
-				(hide yes)
-			)
-		)
-		(property "Description" ""
-			(at 121.92 57.15 0)
-			(effects
-				(font
-					(size 1.27 1.27)
-				)
-				(hide yes)
-			)
-		)
-		(instances
-			(project ""
-				(path "/186d5500-054c-4b47-a89c-85f6ce2abe33"
-					(reference "U3")
-					(unit 1)
-				)
-			)
-		)
-	)
-	(symbol
 		(lib_id "power:+3.3V")
 		(at 222.25 190.5 0)
@@
 	)
 	(symbol
-		(lib_id "Projektin osat:MP2235S")
-		(at 161.29 55.88 0)
-		(unit 1)
-		(exclude_from_sim no)
-		(in_bom yes)
-		(on_board yes)
-		(dnp no)
-		(fields_autoplaced yes)
-		(property "Reference" "U5"
-			(at 162.56 54.6099 0)
-			(effects
-				(font
-					(size 1.27 1.27)
-				)
-				(justify left)
-			)
-		)
-		(property "Value" "~"
-			(at 162.56 57.1499 0)
-			(effects
-				(font
-					(size 1.27 1.27)
-				)
-				(justify left)
-			)
-		)
-		(property "Footprint" ""
-			(at 161.29 55.88 0)
-			(effects
-				(font
-					(size 1.27 1.27)
-				)
-				(hide yes)
-			)
-		)
-		(property "Datasheet" ""
-			(at 161.29 55.88 0)
-			(effects
-				(font
-					(size 1.27 1.27)
-				)
-				(hide yes)
-			)
-		)
-		(property "Description" ""
-			(at 161.29 55.88 0)
-			(effects
-				(font
-					(size 1.27 1.27)
-				)
-				(hide yes)
-			)
-		)
-		(instances
-			(project ""
-				(path "/186d5500-054c-4b47-a89c-85f6ce2abe33"
-					(reference "U5")
-					(unit 1)
-				)
-			)
-		)
-	)
-	(symbol
 		(lib_id "Device:R")
 		(at 25.4 262.89 0)
@@
 	)
 	(symbol
-		(lib_id "Projektin osat:M20048-1")
-		(at 140.97 55.88 0)
+		(lib_id "1_projektin osat:BMP581")
+		(at 105.41 58.42 0)
+		(unit 1)
+		(exclude_from_sim no)
+		(in_bom yes)
+		(on_board yes)
+		(dnp no)
+		(property "Reference" "U3"
+			(at 106.934 57.15 0)
+			(effects
+				(font
+					(size 1.27 1.27)
+				)
+			)
+		)
+		(property "Value" "~"
+			(at 105.41 58.42 0)
+			(effects
+				(font
+					(size 1.27 1.27)
+				)
+				(hide yes)
+			)
+		)
+		(property "Footprint" ""
+			(at 105.41 58.42 0)
+			(effects
+				(font
+					(size 1.27 1.27)
+				)
+				(hide yes)
+			)
+		)
+		(property "Datasheet" ""
+			(at 105.41 58.42 0)
+			(effects
+				(font
+					(size 1.27 1.27)
+				)
+				(hide yes)
+			)
+		)
+		(property "Description" ""
+			(at 105.41 58.42 0)
+			(effects
+				(font
+					(size 1.27 1.27)
+				)
+				(hide yes)
+			)
+		)
+		(pin "4"
+		)
+		(pin "1"
+		)
+		(pin "10"
+		)
+		(pin "3"
+		)
+		(pin "5"
+		)
+		(pin "7"
+		)
+		(pin "9"
+		)
+		(pin "2"
+		)
+		(pin "6"
+		)
+		(pin "8"
+		)
+		(instances
+			(project ""
+				(path "/186d5500-054c-4b47-a89c-85f6ce2abe33"
+					(reference "U3")
+					(unit 1)
+				)
+			)
+		)
+	)
+	(symbol
+		(lib_id "1_projektin osat:M20048-1")
+		(at 149.86 58.42 0)
 		(unit 1)
 		(exclude_from_sim no)
@@
 		(dnp no)
 		(property "Reference" "U4"
-			(at 142.494 53.594 0)
-			(effects
-				(font
-					(size 1.27 1.27)
-				)
-				(justify left)
+			(at 151.384 56.388 0)
+			(effects
+				(font
+					(size 1.27 1.27)
+				)
 			)
 		)
 		(property "Value" "~"
-			(at 142.24 57.1499 0)
-			(effects
-				(font
-					(size 1.27 1.27)
-				)
-				(justify left)
+			(at 149.86 58.42 0)
+			(effects
+				(font
+					(size 1.27 1.27)
+				)
+				(hide yes)
 			)
 		)
 		(property "Footprint" ""
-			(at 140.97 55.88 0)
+			(at 149.86 58.42 0)
 			(effects
 				(font
@@
 		)
 		(property "Datasheet" ""
-			(at 140.97 55.88 0)
+			(at 149.86 58.42 0)
 			(effects
 				(font
@@
 		)
 		(property "Description" ""
-			(at 140.97 55.88 0)
-			(effects
-				(font
-					(size 1.27 1.27)
-				)
-				(hide yes)
-			)
+			(at 149.86 58.42 0)
+			(effects
+				(font
+					(size 1.27 1.27)
+				)
+				(hide yes)
+			)
+		)
+		(pin "24"
+		)
+		(pin "16"
+		)
+		(pin "13"
+		)
+		(pin "4"
+		)
+		(pin "2"
+		)
+		(pin "10"
+		)
+		(pin "6"
+		)
+		(pin "7"
+		)
+		(pin "21"
+		)
+		(pin "5"
+		)
+		(pin "8"
+		)
+		(pin "23"
+		)
+		(pin "19"
+		)
+		(pin "12"
+		)
+		(pin "22"
+		)
+		(pin "9"
+		)
+		(pin "11"
+		)
+		(pin "15"
+		)
+		(pin "17"
+		)
+		(pin "18"
+		)
+		(pin "1"
+		)
+		(pin "28"
+		)
+		(pin "27"
+		)
+		(pin "14"
+		)
+		(pin "26"
+		)
+		(pin "3"
+		)
+		(pin "25"
+		)
+		(pin "20"
 		)
 		(instances
@@
 					(unit 1)
 				)
+			)
+		)
+	)
+	(symbol
+		(lib_id "1_projektin osat:MP2235S")
+		(at 107.95 95.25 0)
+		(unit 1)
+		(exclude_from_sim no)
+		(in_bom yes)
+		(on_board yes)
+		(dnp no)
+		(property "Reference" "U5"
+			(at 109.474 93.98 0)
+			(effects
+				(font
+					(size 1.27 1.27)
+				)
+			)
+		)
+		(property "Value" "~"
+			(at 107.95 95.25 0)
+			(effects
+				(font
+					(size 1.27 1.27)
+				)
+				(hide yes)
+			)
+		)
+		(property "Footprint" ""
+			(at 107.95 95.25 0)
+			(effects
+				(font
+					(size 1.27 1.27)
+				)
+				(hide yes)
+			)
+		)
+		(property "Datasheet" ""
+			(at 107.95 95.25 0)
+			(effects
+				(font
+					(size 1.27 1.27)
+				)
+				(hide yes)
+			)
+		)
+		(property "Description" ""
+			(at 107.95 95.25 0)
+			(effects
+				(font
+					(size 1.27 1.27)
+				)
+				(hide yes)
+			)
+		)
+		(pin "1"
+		)
+		(pin "2"
+		)
+		(pin "3"
+		)
+		(pin "4"
+		)
+		(pin "6"
+		)
+		(pin "8"
+		)
+		(pin "5"
+		)
+		(pin "7"
+		)
+		(instances
+			(project ""
+				(path "/186d5500-054c-4b47-a89c-85f6ce2abe33"
+					(reference "U5")
+					(unit 1)
+				)
