File: KiCad_files/esp.kicad_sch (KiCad schematic)
At the start: 0 parts

Commit message: taikinointia
Other:
- sheet 1_power_supply ports: added none; removed BAT, BAT_STAT
Changed lines of the file:
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@@
-			)
-		)
-		(pin "BAT_STAT" output
-			(at 256.54 100.33 180)
-			(effects
-				(font
-					(size 1.27 1.27)
-				)
-				(justify left)
-			)
-		)
-		(pin "BAT" input
-			(at 256.54 110.49 180)
-			(effects
-				(font
-					(size 1.27 1.27)
-				)
-				(justify left)
 			)
 		)

Commit message: pin header
Other:
- added sheet 1_pin_header (pin_header.kicad_sch)
- sheet 1_power_supply ports: added BAT, BAT_STAT; removed none
Changed lines of the file:
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@@
+	(wire
+		(pts
+			(xy 229.87 181.61) (xy 246.38 181.61)
+		)
+		(stroke
+			(width 0)
+			(type default)
+		)
+	)
+	(wire
+		(pts
+			(xy 246.38 181.61) (xy 246.38 114.3)
+		)
+		(stroke
+			(width 0)
+			(type default)
+		)
+	)
+	(wire
+		(pts
+			(xy 246.38 114.3) (xy 256.54 114.3)
+		)
+		(stroke
+			(width 0)
+			(type default)
+		)
+	)
 	(wire
 		(pts
@@
 			)
 		)
+		(pin "BAT_STAT" output
+			(at 256.54 100.33 180)
+			(effects
+				(font
+					(size 1.27 1.27)
+				)
+				(justify left)
+			)
+		)
+		(pin "BAT" input
+			(at 256.54 114.3 180)
+			(effects
+				(font
+					(size 1.27 1.27)
+				)
+				(justify left)
+			)
+		)
 		(instances
 			(project "esp"
@@
 				)
 			)
+		)
+	)
+	(sheet
+		(at 190.5 154.94)
+		(size 39.37 35.56)
+		(exclude_from_sim no)
+		(in_bom yes)
+		(on_board yes)
+		(dnp no)
+		(fields_autoplaced yes)
+		(stroke
+			(width 0.1524)
+			(type solid)
+		)
+		(fill
+			(color 0 0 0 0.0000)
+		)
+		(property "Sheetname" "1_pin_header"
+			(at 190.5 154.2284 0)
+			(effects
+				(font
+					(size 1.27 1.27)
+				)
+				(justify left bottom)
+			)
+		)
+		(property "Sheetfile" "pin_header.kicad_sch"
+			(at 190.5 191.0846 0)
+			(effects
+				(font
+					(size 1.27 1.27)
+				)
+				(justify left top)
+			)
+		)
+		(pin "PWM3" input
+			(at 229.87 161.29 0)
+			(effects
+				(font
+					(size 1.27 1.27)
+				)
+				(justify right)
+			)
+		)
+		(pin "PWM1" input
+			(at 229.87 168.91 0)
+			(effects
+				(font
+					(size 1.27 1.27)
+				)
+				(justify right)
+			)
+		)
+		(pin "BAT" output
+			(at 229.87 181.61 0)
+			(effects
+				(font
+					(size 1.27 1.27)
+				)
+				(justify right)
+			)
+		)
+		(pin "PWM2" input
+			(at 229.87 165.1 0)
+			(effects
+				(font
+					(size 1.27 1.27)
+				)
+				(justify right)
+			)
+		)
+		(pin "PWM0" input
+			(at 229.87 172.72 0)
+			(effects
+				(font
+					(size 1.27 1.27)
+				)
+				(justify right)
+			)
+		)
+		(instances
+			(project "esp"
+				(path "/186d5500-054c-4b47-a89c-85f6ce2abe33"
+					(page "8")
+				)
+			)

Commit message: i2c
Other:
- sheet 1_IMU ports: added BNO_BOOTN, BNO_CLKSFI0, BNO_NRST, HOST_INTN, HOST_SCL, HOST_SDA; removed none
- sheet 1_MCU ports: added BAROMETER_INT, I2C_CLK, I2C_SDA; removed none

Commit message: välipusku
Other:
- sheet 1_MCU ports: added IMU_INT; removed none
Changed lines of the file:
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@@
 	(wire
 		(pts
-			(xy 195.58 166.37) (xy 208.28 166.37)
+			(xy 189.23 166.37) (xy 208.28 166.37)
 		)
 		(stroke
@@
 	(wire
 		(pts
-			(xy 307.34 140.97) (xy 317.5 140.97)
+			(xy 300.99 140.97) (xy 317.5 140.97)
 		)
 		(stroke
@@
 	(wire
 		(pts
-			(xy 318.77 90.17) (xy 307.34 90.17)
-		)
-		(stroke
-			(width 0)
-			(type default)
-		)
-	)
-	(wire
-		(pts
-			(xy 307.34 146.05) (xy 317.5 146.05)
-		)
-		(stroke
-			(width 0)
-			(type default)
-		)
-	)
-	(wire
-		(pts
-			(xy 307.34 93.98) (xy 318.77 93.98)
-		)
-		(stroke
-			(width 0)
-			(type default)
-		)
-	)
-	(wire
-		(pts
-			(xy 195.58 149.86) (xy 208.28 149.86)
-		)
-		(stroke
-			(width 0)
-			(type default)
-		)
-	)
-	(wire
-		(pts
-			(xy 208.28 146.05) (xy 195.58 146.05)
+			(xy 318.77 90.17) (xy 299.72 90.17)
+		)
+		(stroke
+			(width 0)
+			(type default)
+		)
+	)
+	(wire
+		(pts
+			(xy 300.99 146.05) (xy 317.5 146.05)
+		)
+		(stroke
+			(width 0)
+			(type default)
+		)
+	)
+	(wire
+		(pts
+			(xy 299.72 93.98) (xy 318.77 93.98)
+		)
+		(stroke
+			(width 0)
+			(type default)
+		)
+	)
+	(wire
+		(pts
+			(xy 189.23 149.86) (xy 208.28 149.86)
+		)
+		(stroke
+			(width 0)
+			(type default)
+		)
+	)
+	(wire
+		(pts
+			(xy 208.28 146.05) (xy 189.23 146.05)
 		)
 		(stroke
@@
 	(wire
 		(pts
+			(xy 317.5 149.86) (xy 300.99 149.86)
+		)
+		(stroke
+			(width 0)
+			(type default)
+		)
+	)
+	(wire
+		(pts
 			(xy 91.44 152.4) (xy 107.95 152.4)
 		)
@@
 	(wire
 		(pts
-			(xy 307.34 86.36) (xy 318.77 86.36)
+			(xy 189.23 162.56) (xy 208.28 162.56)
+		)
+		(stroke
+			(width 0)
+			(type default)
+		)
+	)
+	(wire
+		(pts
+			(xy 299.72 86.36) (xy 318.77 86.36)
 		)
 		(stroke
@@
 	)
 	(label "BAROMETER_INT"
-		(at 307.34 93.98 0)
+		(at 299.72 93.98 0)
 		(effects
 			(font
@@
 	)
 	(label "I2C_CLK"
-		(at 307.34 90.17 0)
+		(at 299.72 90.17 0)
 		(effects
 			(font
@@
 	)
 	(label "USB_D-"
-		(at 195.58 149.86 0)
+		(at 189.23 149.86 0)
 		(effects
 			(font
@@
 	)
 	(label "BAROMETER_INT"
-		(at 195.58 166.37 0)
+		(at 189.23 166.37 0)
 		(effects
 			(font
@@
 	)
 	(label "I2C_SDA"
-		(at 307.34 86.36 0)
+		(at 299.72 86.36 0)
 		(effects
 			(font
@@
 	)
 	(label "I2C_CLK"
-		(at 307.34 146.05 0)
+		(at 300.99 146.05 0)
 		(effects
 			(font
@@
 	)
 	(label "USB_D+"
-		(at 195.58 146.05 0)
+		(at 189.23 146.05 0)
+		(effects
+			(font
+				(size 1.27 1.27)
+			)
+			(justify left bottom)
+		)
+	)
+	(label "IMU_INT"
+		(at 189.23 162.56 0)
+		(effects
+			(font
+				(size 1.27 1.27)
+			)
+			(justify left bottom)
+		)
+	)
+	(label "IMU_INT"
+		(at 300.99 149.86 0)
 		(effects
 			(font
@@
 	)
 	(label "I2C_SDA"
-		(at 307.34 140.97 0)
+		(at 300.99 140.97 0)
 		(effects
 			(font
@@
 			)
 		)
-		(pin "HOST_INTN" input
-			(at 317.5 149.86 180)
-			(effects
-				(font
-					(size 1.27 1.27)
-				)
-				(justify left)
-			)
-		)
 		(pin "HOST_SCL" input
 			(at 317.5 146.05 180)
@@
 		(pin "HOST_SDA" bidirectional
 			(at 317.5 140.97 180)
+			(effects
+				(font
+					(size 1.27 1.27)
+				)
+				(justify left)
+			)
+		)
+		(pin "HOST_INTN" output
+			(at 317.5 149.86 180)
 			(effects
 				(font
@@
 	)
 	(sheet
-		(at 208.28 134.62)
-		(size 41.91 36.83)
+		(at 208.28 129.54)
+		(size 41.91 41.91)
 		(exclude_from_sim no)
 		(in_bom yes)
@@
 		)
 		(property "Sheetname" "1_MCU"
-			(at 208.28 133.9084 0)
+			(at 208.28 128.8284 0)
 			(effects
 				(font
@@
 			(effects
 				(font
+					(size 1.27 1.27)
+				)
+				(justify left)
+			)
+		)
+		(pin "IMU_INT" input
+			(at 208.28 162.56 180)
+			(effects
+				(font

Commit message: imu johot
Other:
- sheet 1_IMU ports: added none; removed BNO_CLKSFI0
- sheet 1_MCU ports: added IMU_BOOTN, IMU_NRST; removed none
Changed lines of the file:
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@@
+	(wire
+		(pts
+			(xy 300.99 157.48) (xy 317.5 157.48)
+		)
+		(stroke
+			(width 0)
+			(type default)
+		)
+	)
 	(wire
 		(pts
@@
 	(wire
 		(pts
+			(xy 250.19 152.4) (xy 259.08 152.4)
+		)
+		(stroke
+			(width 0)
+			(type default)
+		)
+	)
+	(wire
+		(pts
 			(xy 250.19 166.37) (xy 259.08 166.37)
 		)
@@
 	(wire
 		(pts
+			(xy 250.19 156.21) (xy 259.08 156.21)
+		)
+		(stroke
+			(width 0)
+			(type default)
+		)
+	)
+	(wire
+		(pts
 			(xy 189.23 149.86) (xy 208.28 149.86)
 		)
@@
 		(pts
 			(xy 250.19 162.56) (xy 259.08 162.56)
+		)
+		(stroke
+			(width 0)
+			(type default)
+		)
+	)
+	(wire
+		(pts
+			(xy 300.99 153.67) (xy 317.5 153.67)
 		)
 		(stroke
@@
 		)
 	)
+	(label "IMU_NRST"
+		(at 259.08 152.4 0)
+		(effects
+			(font
+				(size 1.27 1.27)
+			)
+			(justify left bottom)
+		)
+	)
 	(label "I2C_CLK"
 		(at 299.72 90.17 0)
@@
 		)
 	)
+	(label "IMU_BOOTN"
+		(at 300.99 157.48 0)
+		(effects
+			(font
+				(size 1.27 1.27)
+			)
+			(justify left bottom)
+		)
+	)
+	(label "IMU_BOOTN"
+		(at 259.08 156.21 0)
+		(effects
+			(font
+				(size 1.27 1.27)
+			)
+			(justify left bottom)
+		)
+	)
 	(label "I2C_SDA"
 		(at 299.72 86.36 0)
@@
 	(label "IMU_INT"
 		(at 300.99 149.86 0)
+		(effects
+			(font
+				(size 1.27 1.27)
+			)
+			(justify left bottom)
+		)
+	)
+	(label "IMU_NRST"
+		(at 300.99 153.67 0)
 		(effects
 			(font
@@
 		)
 		(pin "BNO_BOOTN" input
-			(at 317.5 161.29 180)
-			(effects
-				(font
-					(size 1.27 1.27)
-				)
-				(justify left)
-			)
-		)
-		(pin "BNO_CLKSFI0" input
 			(at 317.5 157.48 180)
 			(effects
@@
 			)
 		)
+		(pin "IMU_BOOTN" output
+			(at 250.19 156.21 0)
+			(effects
+				(font
+					(size 1.27 1.27)
+				)
+				(justify right)
+			)
+		)
+		(pin "IMU_NRST" output
+			(at 250.19 152.4 0)
+			(effects
+				(font
+					(size 1.27 1.27)
+				)
+				(justify right)
+			)
+		)

Commit message: puskee
Other:
- sheet 1_GNSS ports: added none; removed E1_BAUD_SELECT, E2_BAUD_SELECT
- sheet 1_MCU ports: added GNSS_FIX, GNSS_HW_R, GNSS_HW_S, GNSS_TM, PWM_0, PWM_1, PWM_2, PWM_3, UART_RX, UART_TX; removed none

Commit message: johtoja
Other:
- sheet 1_MCU ports: added BAT_STAT; removed none
- sheet 1_USB ports: added USB_VBUS; removed none
- sheet 1_power_supply ports: added USB_VBUS; removed none
Changed lines of the file:
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@@
+	(wire
+		(pts
+			(xy 201.93 222.25) (xy 213.36 222.25)
+		)
+		(stroke
+			(width 0)
+			(type default)
+		)
+	)
 	(wire
 		(pts
@@
 	(wire
 		(pts
-			(xy 148.59 226.06) (xy 213.36 226.06)
-		)
-		(stroke
-			(width 0)
-			(type default)
-		)
-	)
-	(wire
-		(pts
 			(xy 303.53 220.98) (xy 318.77 220.98)
 		)
@@
 	(wire
 		(pts
+			(xy 251.46 209.55) (xy 259.08 209.55)
+		)
+		(stroke
+			(width 0)
+			(type default)
+		)
+	)
+	(wire
+		(pts
 			(xy 303.53 218.44) (xy 318.77 218.44)
 		)
@@
 	(wire
 		(pts
+			(xy 201.93 226.06) (xy 213.36 226.06)
+		)
+		(stroke
+			(width 0)
+			(type default)
+		)
+	)
+	(wire
+		(pts
 			(xy 250.19 107.95) (xy 260.35 107.95)
 		)
@@
 	(wire
 		(pts
+			(xy 163.83 148.59) (xy 173.99 148.59)
+		)
+		(stroke
+			(width 0)
+			(type default)
+		)
+	)
+	(wire
+		(pts
 			(xy 250.19 123.19) (xy 260.35 123.19)
 		)
@@
 	(wire
 		(pts
+			(xy 148.59 226.06) (xy 156.21 226.06)
+		)
+		(stroke
+			(width 0)
+			(type default)
+		)
+	)
+	(wire
+		(pts
 			(xy 208.28 146.05) (xy 189.23 146.05)
 		)
@@
 		(pts
 			(xy 91.44 152.4) (xy 107.95 152.4)
+		)
+		(stroke
+			(width 0)
+			(type default)
+		)
+	)
+	(wire
+		(pts
+			(xy 189.23 153.67) (xy 208.28 153.67)
 		)
 		(stroke
@@
 		)
 	)
+	(label "USB_VBUS"
+		(at 173.99 148.59 0)
+		(effects
+			(font
+				(size 1.27 1.27)
+			)
+			(justify left bottom)
+		)
+	)
 	(label "BAROMETER_INT"
 		(at 299.72 93.98 0)
@@
 		)
 	)
+	(label "BAT"
+		(at 156.21 226.06 0)
+		(effects
+			(font
+				(size 1.27 1.27)
+			)
+			(justify left bottom)
+		)
+	)
+	(label "BAT_STAT"
+		(at 189.23 153.67 0)
+		(effects
+			(font
+				(size 1.27 1.27)
+			)
+			(justify left bottom)
+		)
+	)
 	(label "GNSS_TX"
 		(at 260.35 139.7 0)
@@
 		)
 	)
+	(label "BAT_STAT"
+		(at 259.08 209.55 0)
+		(effects
+			(font
+				(size 1.27 1.27)
+			)
+			(justify left bottom)
+		)
+	)
+	(label "BAT"
+		(at 201.93 226.06 0)
+		(effects
+			(font
+				(size 1.27 1.27)
+			)
+			(justify left bottom)
+		)
+	)
 	(label "GNSS_HW_S"
 		(at 303.53 215.9 0)
@@
 		)
 	)
+	(label "USB_VBUS"
+		(at 201.93 222.25 0)
+		(effects
+			(font
+				(size 1.27 1.27)
+			)
+			(justify left bottom)
+		)
+	)
 	(label "GNSS_HW_R"
 		(at 260.35 127 0)
@@
 	(label "GNSS_FIX"
 		(at 303.53 210.82 0)
+		(effects
+			(font
+				(size 1.27 1.27)
+			)
+			(justify left bottom)
+		)
+	)
+	(label ""
+		(at 189.23 125.73 0)
 		(effects
 			(font
@@
 			)
 		)
-		(pin "BAT_STAT" output
-			(at 213.36 212.09 180)
-			(effects
-				(font
-					(size 1.27 1.27)
-				)
-				(justify left)
-			)
-		)
 		(pin "BAT" input
 			(at 213.36 226.06 180)
@@
 				)
 				(justify left)
+			)
+		)
+		(pin "USB_VBUS" input
+			(at 213.36 222.25 180)
+			(effects
+				(font
+					(size 1.27 1.27)
+				)
+				(justify left)
+			)
+		)
+		(pin "BAT_STAT" output
+			(at 251.46 209.55 0)
+			(effects
+				(font
+					(size 1.27 1.27)
+				)
+				(justify right)
 			)
 		)
@@
 			)
 		)
+		(pin "BAT_STAT" input
+			(at 208.28 153.67 180)
+			(effects
+				(font
+					(size 1.27 1.27)
+				)
+				(justify left)
+			)
+		)
 		(instances
 			(project "esp"
@@
 			)
 		)
+		(pin "USB_VBUS" output
+			(at 163.83 148.59 0)
+			(effects
+				(font
+					(size 1.27 1.27)
+				)
+				(justify right)
+			)
+		)
