File: KiCad_files/MCU.kicad_sch (KiCad schematic)
At the start: 6 parts, among them SW2 SW_Push, U12 ESP32-S3-MINI-1U

Commit message: GNSS aloitettu
Changed lines of the file:
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@@
 		)
 	)
-	(label "USB_D+"
+	(hierarchical_label "USB_D-"
+		(shape bidirectional)
+		(at 187.96 87.63 0)
+		(effects
+			(font
+				(size 1.27 1.27)
+			)
+			(justify left)
+		)
+	)
+	(hierarchical_label "USB_D+"
+		(shape bidirectional)
 		(at 187.96 90.17 0)
 		(effects
@@
 				(size 1.27 1.27)
 			)
-			(justify left bottom)
+			(justify left)
 		)
 	)
-	(label "USB_D-"
-		(at 187.96 87.63 0)
-		(effects
-			(font
-				(size 1.27 1.27)
-			)
-			(justify left bottom)
-		)
-	)

Commit message: taikinointia
Parts:
- removed SW2: SW_Push, symbol Switch:SW_Push
- added U1: B3U-1000P, B3U-1000P, symbol 1_projektin osat:B3U-1000P
- C6, C7, C8: footprint (none) -> Capacitor_SMD:C_0805_2012Metric_Pad1.18x1.45mm_HandSolder
- R8: footprint (none) -> Resistor_SMD:R_0805_2012Metric_Pad1.20x1.40mm_HandSolder
Connections:
- net GND: now also U1.1
- net at C6.1, R8.1, U12.45 (EN): now also U1.2
Changed lines of the file:
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@@
 	(text "Hardware reset with RC delay\ncircuit to ensure stable booting"
 		(exclude_from_sim no)
-		(at 110.998 67.31 0)
+		(at 109.982 64.516 0)
 		(effects
 			(font
@@
 	(wire
 		(pts
-			(xy 116.84 80.01) (xy 114.3 80.01)
+			(xy 86.36 80.01) (xy 81.28 80.01)
 		)
 		(stroke
@@
 	(wire
 		(pts
-			(xy 114.3 80.01) (xy 114.3 91.44)
-		)
-		(stroke
-			(width 0)
-			(type default)
-		)
-	)
-	(wire
-		(pts
-			(xy 114.3 91.44) (xy 130.81 91.44)
+			(xy 81.28 80.01) (xy 81.28 91.44)
+		)
+		(stroke
+			(width 0)
+			(type default)
+		)
+	)
+	(wire
+		(pts
+			(xy 81.28 91.44) (xy 130.81 91.44)
 		)
 		(stroke
@@
 			)
 		)
-		(property "Footprint" ""
+		(property "Footprint" "Capacitor_SMD:C_0805_2012Metric_Pad1.18x1.45mm_HandSolder"
 			(at 155.9052 60.96 0)
 			(effects
@@
 			)
 		)
-		(property "Footprint" ""
+		(property "Footprint" "Capacitor_SMD:C_0805_2012Metric_Pad1.18x1.45mm_HandSolder"
 			(at 131.7752 90.17 0)
 			(effects
@@
 			)
 		)
-		(property "Footprint" ""
+		(property "Footprint" "Capacitor_SMD:C_0805_2012Metric_Pad1.18x1.45mm_HandSolder"
 			(at 144.4752 60.96 0)
 			(effects
@@
 	)
 	(symbol
+		(lib_id "1_projektin osat:B3U-1000P")
+		(at 86.36 80.01 0)
+		(unit 1)
+		(exclude_from_sim no)
+		(in_bom yes)
+		(on_board yes)
+		(dnp no)
+		(fields_autoplaced yes)
+		(property "Reference" "U1"
+			(at 106.68 69.85 0)
+			(effects
+				(font
+					(size 1.524 1.524)
+				)
+			)
+		)
+		(property "Value" "B3U-1000P"
+			(at 106.68 72.39 0)
+			(effects
+				(font
+					(size 1.524 1.524)
+				)
+			)
+		)
+		(property "Footprint" "B3U-1000P"
+			(at 86.36 80.01 0)
+			(effects
+				(font
+					(size 1.27 1.27)
+					(italic yes)
+				)
+				(hide yes)
+			)
+		)
+		(property "Datasheet" "B3U-1000P"
+			(at 86.36 80.01 0)
+			(effects
+				(font
+					(size 1.27 1.27)
+					(italic yes)
+				)
+				(hide yes)
+			)
+		)
+		(property "Description" ""
+			(at 86.36 80.01 0)
+			(effects
+				(font
+					(size 1.27 1.27)
+				)
+				(hide yes)
+			)
+		)
+		(pin "1"
+		)
+		(pin "2"
+		)
+		(instances
+			(project ""
+				(path "/186d5500-054c-4b47-a89c-85f6ce2abe33/da295ba5-5e07-44a9-8c1c-e3f6c5500b46"
+					(reference "U1")
+					(unit 1)
+				)
+			)
+		)
+	)
+	(symbol
 		(lib_id "Device:R")
 		(at 130.81 73.66 180)
@@
 			)
 		)
-		(property "Footprint" ""
+		(property "Footprint" "Resistor_SMD:R_0805_2012Metric_Pad1.20x1.40mm_HandSolder"
 			(at 132.588 73.66 90)
 			(effects
@@
 					(unit 1)
 				)
-			)
-		)
-	)
-	(symbol
-		(lib_id "Switch:SW_Push")
-		(at 121.92 80.01 0)
-		(unit 1)
-		(exclude_from_sim no)
-		(in_bom yes)
-		(on_board yes)
-		(dnp no)
-		(fields_autoplaced yes)
-		(property "Reference" "SW2"
-			(at 121.92 72.39 0)
-			(effects
-				(font
-					(size 1.27 1.27)
-				)
-			)
-		)
-		(property "Value" "SW_Push"
-			(at 121.92 74.93 0)
-			(effects
-				(font
-					(size 1.27 1.27)
-				)
-			)
-		)
-		(property "Footprint" ""
-			(at 121.92 74.93 0)
-			(effects
-				(font
-					(size 1.27 1.27)
-				)
-				(hide yes)
-			)
-		)
-		(property "Datasheet" "~"
-			(at 121.92 74.93 0)
-			(effects
-				(font
-					(size 1.27 1.27)
-				)
-				(hide yes)
-			)
-		)
-		(property "Description" "Push button switch, generic, two pins"
-			(at 121.92 80.01 0)
-			(effects
-				(font
-					(size 1.27 1.27)
-				)
-				(hide yes)
-			)
-		)
-		(pin "1"
-		)
-		(pin "2"
-		)
-		(instances
-			(project "esp"
-				(path "/186d5500-054c-4b47-a89c-85f6ce2abe33/da295ba5-5e07-44a9-8c1c-e3f6c5500b46"
-					(reference "SW2")
-					(unit 1)
-				)

Commit message: ajan tasalle
Parts:
- U1: DigiKey (none) -> SW1020CT-ND
Changed lines of the file:
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@@
+			)
+		)
+		(property "DigiKey" "SW1020CT-ND"
+			(at 86.36 80.01 0)
+			(effects
+				(font
+					(size 1.27 1.27)
+				)
+				(hide yes)
 			)
 		)

Commit message: välipusku
Changed lines of the file:
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@@
+		)
+	)
+	(hierarchical_label "IMU_INT"
+		(shape input)
+		(at 204.47 132.08 0)
+		(effects
+			(font
+				(size 1.27 1.27)
+			)
+			(justify left)
 		)
 	)

Commit message: imu johot
Changed lines of the file:
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@@
 	(hierarchical_label "BAROMETER_INT"
 		(shape input)
-		(at 204.47 127 0)
+		(at 205.74 121.92 0)
+		(effects
+			(font
+				(size 1.27 1.27)
+			)
+			(justify left)
+		)
+	)
+	(hierarchical_label "IMU_BOOTN"
+		(shape output)
+		(at 205.74 135.89 0)
 		(effects
 			(font
@@
 	(hierarchical_label "I2C_SDA"
 		(shape bidirectional)
-		(at 205.74 113.03 0)
+		(at 205.74 114.3 0)
 		(effects
 			(font
@@
 	(hierarchical_label "IMU_INT"
 		(shape input)
-		(at 204.47 132.08 0)
+		(at 205.74 125.73 0)
 		(effects
 			(font
+				(size 1.27 1.27)
+			)
+			(justify left)
+		)
+	)
+	(hierarchical_label "IMU_NRST"
+		(shape output)
+		(at 205.74 130.81 0)
+		(effects
+			(font

Commit message: sdfasa
Parts:
- C6: DigiKey (none) -> 720-1754-1-ND
- C7: value 1u -> 2.2u; DigiKey (none) -> 399-C0805C225K4RACTUCT-ND
- C8: value 10n -> 0.1u; DigiKey (none) -> 720-1754-1-ND
- R8: DigiKey (none) -> 541-10.0KCCT-ND
- U12: DigiKey (none) -> 1965-ESP32-S3-MINI-1U-N8CT-ND
Changed lines of the file:
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@@
 			)
 		)
-		(property "Value" "10n"
+		(property "Value" "0.1u"
 			(at 158.75 58.4199 0)
 			(effects
@@
 			)
 		)
+		(property "DigiKey" "720-1754-1-ND"
+			(at 154.94 57.15 0)
+			(effects
+				(font
+					(size 1.27 1.27)
+				)
+				(hide yes)
+			)
+		)
 		(pin "2"
 		)
@@
 			)
 		)
+		(property "DigiKey" "720-1754-1-ND"
+			(at 130.81 86.36 0)
+			(effects
+				(font
+					(size 1.27 1.27)
+				)
+				(hide yes)
+			)
+		)
 		(pin "1"
 		)
@@
 			)
 		)
-		(property "Value" "1u"
+		(property "Value" "2.2u"
 			(at 147.32 58.4199 0)
 			(effects
@@
 			)
 		)
+		(property "DigiKey" "399-C0805C225K4RACTUCT-ND"
+			(at 143.51 57.15 0)
+			(effects
+				(font
+					(size 1.27 1.27)
+				)
+				(hide yes)
+			)
+		)
 		(pin "2"
 		)
@@
 			)
 		)
+		(property "DigiKey" "541-10.0KCCT-ND"
+			(at 130.81 73.66 0)
+			(effects
+				(font
+					(size 1.27 1.27)
+				)
+				(hide yes)
+			)
+		)
 		(pin "2"
 		)
@@
 			(at 166.37 105.41 0)
 			(effects
+				(font
+					(size 1.27 1.27)
+				)
+				(hide yes)
+			)
+		)
+		(property "DigiKey" "1965-ESP32-S3-MINI-1U-N8CT-ND"
+			(at 166.37 105.41 0)
+			(effects
