File: KiCad_files/barometer.kicad_sch (KiCad schematic)
At the start: 1 part

Commit message: barometri
Parts:
- added C15, C16: 100n, symbol Device:C
Connections:
- net +3.3V: now reaches U11.1 (VDD_IO)
- net +3.3V: now also U11.10 (VDD), U11.6 (CSB), C15.1, C16.1
- net SCK: now reaches U11.2 (SCK)
- net GND: now reaches U11.3 (VSS)
- net GND: now also U11.7 (INT), U11.8 (VSS), U11.9 (VSS), C15.2, C16.2
- net SDI: now reaches U11.4 (SDI)
- net SDO: now reaches U11.5 (SDO)
Other:
- note added: "All VSS pins must be connected to the ground."
- note added: "Chip select pin(CSB) should be connected to VCC in order to start serial interface in I2C mode."
- note added: "Interrupt pin(INT) should be connected to the ground if not used. See page 46 section 6.2 from the datasheet."

Commit message: barometri
Connections:
- net SDO is gone; now on net GND: U11.5 (SDO)
Other:
- note added: "The I2C slave address of BMP581 is 7'h46 for SDO = 1'b0 and 7'h47 for SDO = 1'b1."
Changed lines of the file:
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@@
+		)
+	)
+	(text "The I2C slave address of BMP581 is 7'h46 for SDO = 1'b0 and 7'h47 for SDO = 1'b1."
+		(exclude_from_sim no)
+		(at 192.024 88.138 0)
+		(effects
+			(font
+				(size 1.27 1.27)
+			)
 		)
 	)
@@
 	(wire
 		(pts
-			(xy 144.78 92.71) (xy 149.86 92.71)
+			(xy 144.78 92.71) (xy 153.67 92.71)
 		)
 		(stroke
@@
 	)
 	(hierarchical_label "SDI"
-		(shape input)
+		(shape bidirectional)
 		(at 110.49 95.25 180)
 		(effects
@@
 		)
 	)
-	(hierarchical_label "SDO"
-		(shape input)
-		(at 149.86 92.71 0)
-		(effects
-			(font
-				(size 1.27 1.27)
-			)
-			(justify left)
-		)
-	)
+	(symbol
+		(lib_id "power:GND")
+		(at 153.67 92.71 90)
+		(unit 1)
+		(exclude_from_sim no)
+		(in_bom yes)
+		(on_board yes)
+		(dnp no)
+		(fields_autoplaced yes)
+		(property "Reference" "#PWR048"
+			(at 160.02 92.71 0)
+			(effects
+				(font
+					(size 1.27 1.27)
+				)
+				(hide yes)
+			)
+		)
+		(property "Value" "GND"
+			(at 157.48 92.7099 90)
+			(effects
+				(font
+					(size 1.27 1.27)
+				)
+				(justify right)
+			)
+		)
+		(property "Footprint" ""
+			(at 153.67 92.71 0)
+			(effects
+				(font
+					(size 1.27 1.27)
+				)
+				(hide yes)
+			)
+		)
+		(property "Datasheet" ""
+			(at 153.67 92.71 0)
+			(effects
+				(font
+					(size 1.27 1.27)
+				)
+				(hide yes)
+			)
+		)
+		(property "Description" "Power symbol creates a global label with name \"GND\" , ground"
+			(at 153.67 92.71 0)
+			(effects
+				(font
+					(size 1.27 1.27)
+				)
+				(hide yes)
+			)
+		)
+		(pin "1"
+		)
+		(instances
+			(project ""
+				(path "/186d5500-054c-4b47-a89c-85f6ce2abe33/117263c6-b09f-4555-b324-57dde8b40725"
+					(reference "#PWR048")
+					(unit 1)
+				)
+			)
+		)
+	)

Commit message: interrupt output
Connections:
- net GND: no longer U11.7 (INT)
- new net INT: U11.7 (INT)
Changed lines of the file:
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@@
 	(text "The I2C slave address of BMP581 is 7'h46 for SDO = 1'b0 and 7'h47 for SDO = 1'b1."
 		(exclude_from_sim no)
-		(at 192.024 88.138 0)
+		(at 202.184 87.884 0)
 		(effects
 			(font
@@
 	(text "Interrupt pin(INT) should be connected to the ground if not used.\nSee page 46 section 6.2 from the datasheet."
 		(exclude_from_sim no)
-		(at 182.118 99.822 0)
+		(at 192.532 99.822 0)
 		(effects
 			(font
@@
 	(wire
 		(pts
-			(xy 144.78 97.79) (xy 148.59 97.79)
+			(xy 144.78 97.79) (xy 154.94 97.79)
 		)
 		(stroke
@@
 		(pts
 			(xy 129.54 107.95) (xy 129.54 111.76)
-		)
-		(stroke
-			(width 0)
-			(type default)
-		)
-	)
-	(wire
-		(pts
-			(xy 148.59 97.79) (xy 148.59 116.84)
 		)
 		(stroke
@@
 		)
 	)
+	(hierarchical_label "INT"
+		(shape output)
+		(at 154.94 97.79 0)
+		(effects
+			(font
+				(size 1.27 1.27)
+			)
+			(justify left)
+		)
+	)
 	(symbol
 		(lib_id "power:GND")
@@
 					(unit 1)
 				)
-			)
-		)
-	)
-	(symbol
-		(lib_id "power:GND")
-		(at 148.59 116.84 0)
-		(unit 1)
-		(exclude_from_sim no)
-		(in_bom yes)
-		(on_board yes)
-		(dnp no)
-		(fields_autoplaced yes)
-		(property "Reference" "#PWR042"
-			(at 148.59 123.19 0)
-			(effects
-				(font
-					(size 1.27 1.27)
-				)
-				(hide yes)
-			)
-		)
-		(property "Value" "GND"
-			(at 148.59 121.92 0)
-			(effects
-				(font
-					(size 1.27 1.27)
-				)
-			)
-		)
-		(property "Footprint" ""
-			(at 148.59 116.84 0)
-			(effects
-				(font
-					(size 1.27 1.27)
-				)
-				(hide yes)
-			)
-		)
-		(property "Datasheet" ""
-			(at 148.59 116.84 0)
-			(effects
-				(font
-					(size 1.27 1.27)
-				)
-				(hide yes)
-			)
-		)
-		(property "Description" "Power symbol creates a global label with name \"GND\" , ground"
-			(at 148.59 116.84 0)
-			(effects
-				(font
-					(size 1.27 1.27)
-				)
-				(hide yes)
-			)
-		)
-		(pin "1"
-		)
-		(instances
-			(project "esp"
-				(path "/186d5500-054c-4b47-a89c-85f6ce2abe33/117263c6-b09f-4555-b324-57dde8b40725"
-					(reference "#PWR042")
-					(unit 1)
-				)

Commit message: footprinttejä
Parts:
- C15, C16: value 100n -> 0.1u
- U11: footprint (none) -> 1_project_library:QFN10_BMP581_BOS
Changed lines of the file:
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@@
 			)
 		)
-		(property "Value" "100n"
+		(property "Value" "0.1u"
 			(at 119.38 74.9299 0)
 			(effects
@@
 			)
 		)
-		(property "Footprint" ""
+		(property "Footprint" "1_project_library:QFN10_BMP581_BOS"
 			(at 121.92 85.09 0)
 			(effects
@@
 			)
 		)
-		(property "Value" "100n"
+		(property "Value" "0.1u"
 			(at 149.86 74.9299 0)
 			(effects

Commit message: update
Parts:
- C15, C16: DigiKey (none) -> 720-1754-1-ND
- U11: DigiKey (none) -> 828-BMP581CT-ND
Changed lines of the file:
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@@
+			)
+		)
+		(property "DigiKey" "720-1754-1-ND"
+			(at 115.57 73.66 0)
+			(effects
+				(font
+					(size 1.27 1.27)
+				)
+				(hide yes)
 			)
 		)
@@
 			)
 		)
+		(property "DigiKey" "828-BMP581CT-ND"
+			(at 121.92 85.09 0)
+			(effects
+				(font
+					(size 1.27 1.27)
+				)
+				(hide yes)
+			)
+		)
 		(pin "4"
 		)
@@
 			(at 146.05 73.66 0)
 			(effects
+				(font
+					(size 1.27 1.27)
+				)
+				(hide yes)
+			)
+		)
+		(property "DigiKey" "720-1754-1-ND"
+			(at 146.05 73.66 0)
+			(effects

Commit message: sdfasa
Parts:
- C15, C16: footprint (none) -> Capacitor_SMD:C_0805_2012Metric_Pad1.18x1.45mm_HandSolder
Changed lines of the file:
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@@
 			)
 		)
-		(property "Footprint" ""
+		(property "Footprint" "Capacitor_SMD:C_0805_2012Metric_Pad1.18x1.45mm_HandSolder"
 			(at 116.5352 77.47 0)
 			(effects
@@
 			)
 		)
-		(property "Footprint" ""
+		(property "Footprint" "Capacitor_SMD:C_0805_2012Metric_Pad1.18x1.45mm_HandSolder"
 			(at 147.0152 77.47 0)
 			(effects
