File: KiCad_files/GNSS.kicad_sch (KiCad schematic)
At the start: 12 parts, among them U2 1060

Commit message: puskee
Connections:
- net E1_BAUD_SELECT: no longer names the net of U10.13 (E2)
- net E2_BAUD_SELECT: no longer names the net of U10.14 (E3)
- no-connect marks 0 -> 2
Changed lines of the file:
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@@
 		(color 0 0 0 0)
 	)
+	(no_connect
+		(at 71.12 151.13)
+	)
+	(no_connect
+		(at 67.31 148.59)
+	)
 	(wire
 		(pts
@@
 	(wire
 		(pts
+			(xy 129.54 116.84) (xy 129.54 148.59)
+		)
+		(stroke
+			(width 0)
+			(type default)
+		)
+	)
+	(wire
+		(pts
 			(xy 203.2 104.14) (xy 215.9 104.14)
 		)
@@
 	(wire
 		(pts
+			(xy 132.08 116.84) (xy 132.08 151.13)
+		)
+		(stroke
+			(width 0)
+			(type default)
+		)
+	)
+	(wire
+		(pts
 			(xy 76.2 63.5) (xy 76.2 101.6)
 		)
@@
 	(wire
 		(pts
+			(xy 71.12 151.13) (xy 132.08 151.13)
+		)
+		(stroke
+			(width 0)
+			(type default)
+		)
+	)
+	(wire
+		(pts
 			(xy 81.28 167.64) (xy 81.28 180.34)
 		)
@@
 	(wire
 		(pts
-			(xy 132.08 116.84) (xy 132.08 153.67)
-		)
-		(stroke
-			(width 0)
-			(type default)
-		)
-	)
-	(wire
-		(pts
 			(xy 134.62 123.19) (xy 160.02 123.19)
 		)
@@
 	(wire
 		(pts
-			(xy 50.8 151.13) (xy 129.54 151.13)
-		)
-		(stroke
-			(width 0)
-			(type default)
-		)
-	)
-	(wire
-		(pts
 			(xy 173.99 62.23) (xy 177.8 62.23)
 		)
@@
 	(wire
 		(pts
-			(xy 50.8 153.67) (xy 132.08 153.67)
-		)
-		(stroke
-			(width 0)
-			(type default)
-		)
-	)
-	(wire
-		(pts
 			(xy 156.21 106.68) (xy 160.02 106.68)
 		)
@@
 	(wire
 		(pts
-			(xy 129.54 116.84) (xy 129.54 151.13)
-		)
-		(stroke
-			(width 0)
-			(type default)
-		)
-	)
-	(wire
-		(pts
 			(xy 106.68 62.23) (xy 99.06 62.23)
 		)
@@
 		(pts
 			(xy 160.02 99.06) (xy 160.02 96.52)
+		)
+		(stroke
+			(width 0)
+			(type default)
+		)
+	)
+	(wire
+		(pts
+			(xy 67.31 148.59) (xy 129.54 148.59)
 		)
 		(stroke
@@
 		(effects
 			(font
-				(size 1.27 1.27)
-			)
-			(justify right)
-		)
-	)
-	(hierarchical_label "E2_BAUD_SELECT"
-		(shape input)
-		(at 50.8 153.67 180)
-		(effects
-			(font
-				(size 1.27 1.27)
-			)
-			(justify right)
-		)
-	)
-	(hierarchical_label "E1_BAUD_SELECT"
-		(shape input)
-		(at 50.8 151.13 180)
-		(effects
-			(font

Commit message: pwr_flags
Changed lines of the file:
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@@
+	)
+	(junction
+		(at 121.92 167.64)
+		(diameter 0)
+		(color 0 0 0 0)
 	)
 	(junction
@@
 		)
 	)
+	(symbol
+		(lib_id "power:PWR_FLAG")
+		(at 121.92 167.64 0)
+		(unit 1)
+		(exclude_from_sim no)
+		(in_bom yes)
+		(on_board yes)
+		(dnp no)
+		(fields_autoplaced yes)
+		(property "Reference" "#FLG03"
+			(at 121.92 165.735 0)
+			(effects
+				(font
+					(size 1.27 1.27)
+				)
+				(hide yes)
+			)
+		)
+		(property "Value" "PWR_FLAG"
+			(at 121.92 162.56 0)
+			(effects
+				(font
+					(size 1.27 1.27)
+				)
+			)
+		)
+		(property "Footprint" ""
+			(at 121.92 167.64 0)
+			(effects
+				(font
+					(size 1.27 1.27)
+				)
+				(hide yes)
+			)
+		)
+		(property "Datasheet" "~"
+			(at 121.92 167.64 0)
+			(effects
+				(font
+					(size 1.27 1.27)
+				)
+				(hide yes)
+			)
+		)
+		(property "Description" "Special symbol for telling ERC where power comes from"
+			(at 121.92 167.64 0)
+			(effects
+				(font
+					(size 1.27 1.27)
+				)
+				(hide yes)
+			)
+		)
+		(pin "1"
+		)
+		(instances
+			(project ""
+				(path "/186d5500-054c-4b47-a89c-85f6ce2abe33/58061273-0348-4c5f-98ae-c78a02c73d37"
+					(reference "#FLG03")
+					(unit 1)
+				)
+			)
+		)
+	)
