File: KiCad_files/powersupply.kicad_pcb (KiCad board)
At the start: 2 copper layers, 61 parts, among them J1 Conn_01x08_Socket, J2 USB4105-GF-A, Q2 DMP3099L, SW1 SLW-171175-7A-N-D, U1 B3U-1000P, U12 ESP32-S3-MINI-1U, U13 BNO085, U2 1060, U7 LTC4412xS6

Commit message: powersupply pcb
Parts:
- moved C17 28.6 mm to (58.5, 135.1)
- moved U8 28.6 mm to (57.1, 131.1)
- moved C19 28.6 mm to (62.0, 123.7)
- moved C20 28.6 mm to (55.0, 135.0)
- moved C25 28.6 mm to (73.0, 133.1)
- moved C27 28.6 mm to (76.5, 133.1)
- moved D1 28.6 mm to (73.0, 123.6)
- moved L4 28.6 mm to (65.5, 131.7)
- moved Q2 28.6 mm to (43.6, 129.2)
- moved R1 28.6 mm to (73.0, 127.6)
- moved R10 28.6 mm to (55.1, 126.7)
- moved R11 28.6 mm to (58.0, 123.7)
- moved R14 28.6 mm to (58.5, 119.7)
- moved R15 28.6 mm to (80.5, 132.6)
- moved C18 28.6 mm to (51.5, 127.1)
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Routing:
- net GND: track 123.6 -> 108.9 mm, vias 5 -> 4
- net Net-(Q2-D): track 15.0 -> 17.6 mm
- net Net-(U8-SW): track 12.7 -> 10.8 mm
- net +3.3V: track 34.0 -> 33.0 mm
- net Net-(D2-K): track 28.3 -> 27.5 mm
- net Net-(U8-EN/SYNC): track 5.82 -> 5.15 mm
- added copper zone on F.Cu, net (none)
- added copper zone on B.Cu, net GND
Other:
- board outline added: 100 x 100 mm
